File: hw/pcb/impl/senseye-insight/stonyman-breakout-adc.sch (EAGLE design)
At the start: 8 parts

Commit message: finished routing the ADC connector boards
it seems to have passed the "ERC" check, but I didn't do a DRC.  I
haven't verified that it is the correct size yet.  And, I might change
some of the routing
Parts:
- JP1: value M12LOCK_LONGPADS -> M12PTH; device SparkFun:M12LOCK_LONGPADS -> SparkFun-Connectors:M12PTH
- JP2: value M09LOCK -> M09; device SparkFun:M09LOCK -> SparkFun-Connectors:M09
Changed lines of the file:
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@@
 <layer number="106" name="bPlate" color="7" fill="1" visible="no" active="yes"/>
 <layer number="107" name="Crop" color="7" fill="1" visible="no" active="yes"/>
+<layer number="108" name="tplace-old" color="10" fill="1" visible="yes" active="yes"/>
+<layer number="109" name="ref-old" color="11" fill="1" visible="yes" active="yes"/>
 <layer number="116" name="Patch_BOT" color="9" fill="4" visible="no" active="yes"/>
 <layer number="121" name="_tsilk" color="7" fill="1" visible="no" active="yes"/>
@@
 <layer number="144" name="Drill_legend" color="7" fill="1" visible="no" active="yes"/>
 <layer number="151" name="HeatSink" color="7" fill="1" visible="no" active="yes"/>
+<layer number="199" name="Contour" color="7" fill="1" visible="yes" active="yes"/>
 <layer number="200" name="200bmp" color="1" fill="10" visible="no" active="yes"/>
 <layer number="201" name="201bmp" color="2" fill="10" visible="no" active="yes"/>
@@
 </classes>
 <parts>
-<part name="JP1" library="SparkFun" deviceset="M12" device="LOCK_LONGPADS"/>
-<part name="JP2" library="SparkFun" deviceset="M09" device="LOCK"/>
 <part name="U$1" library="senseye" deviceset="TI_ADC081S101" device=""/>
 <part name="C1" library="rcl" deviceset="C-EU" device="C0603" value="1nF"/>
@@
 <part name="C4" library="rcl" deviceset="C-EU" device="C0603" value="1uF"/>
 <part name="R1" library="rcl" deviceset="R-US_" device="R0603" value="0 or UNPOP"/>
+<part name="JP1" library="SparkFun-Connectors" deviceset="M12" device="PTH"/>
+<part name="JP2" library="SparkFun-Connectors" deviceset="M09" device=""/>
 </parts>
 <sheets>
@@
 </plain>
 <instances>
-<instance part="JP1" gate="G$1" x="-2.54" y="38.1"/>
-<instance part="JP2" gate="G$1" x="76.2" y="35.56" rot="R180"/>
 <instance part="U$1" gate="G$1" x="58.42" y="2.54"/>
 <instance part="C1" gate="G$1" x="45.72" y="50.8" rot="R90"/>
@@
 <instance part="C4" gate="G$1" x="35.56" y="0"/>
 <instance part="R1" gate="G$1" x="17.78" y="60.96"/>
+<instance part="JP1" gate="G$1" x="-2.54" y="38.1"/>
+<instance part="JP2" gate="G$1" x="76.2" y="35.56" rot="R180"/>
 </instances>
 <busses>
@@
 <net name="GND" class="0">
 <segment>
-<pinref part="JP1" gate="G$1" pin="10"/>
-<pinref part="JP2" gate="G$1" pin="1"/>
 <wire x1="7.62" y1="45.72" x2="25.4" y2="45.72" width="0.1524" layer="91"/>
 <label x="10.16" y="45.72" size="1.778" layer="95"/>
@@
 <junction x="35.56" y="2.54"/>
 <pinref part="U$1" gate="G$1" pin="GND"/>
+<pinref part="JP1" gate="G$1" pin="10"/>
+<pinref part="JP2" gate="G$1" pin="1"/>
 </segment>
 </net>
 <net name="V_STONY" class="0">
 <segment>
-<pinref part="JP1" gate="G$1" pin="9"/>
-<pinref part="JP2" gate="G$1" pin="2"/>
 <wire x1="7.62" y1="43.18" x2="43.18" y2="43.18" width="0.1524" layer="91"/>
 <label x="10.16" y="43.18" size="1.778" layer="95"/>
@@
 <wire x1="43.18" y1="50.8" x2="43.18" y2="43.18" width="0.1524" layer="91"/>
 <junction x="43.18" y="43.18"/>
+<pinref part="JP1" gate="G$1" pin="9"/>
+<pinref part="JP2" gate="G$1" pin="2"/>
 </segment>
 <segment>
@@
 <net name="RESP" class="0">
 <segment>
-<pinref part="JP2" gate="G$1" pin="3"/>
-<pinref part="JP1" gate="G$1" pin="8"/>
 <wire x1="66.04" y1="40.64" x2="7.62" y2="40.64" width="0.1524" layer="91"/>
 <label x="10.16" y="40.64" size="1.778" layer="95"/>
+<pinref part="JP1" gate="G$1" pin="8"/>
+<pinref part="JP2" gate="G$1" pin="3"/>
 </segment>
 </net>
 <net name="INCP" class="0">
 <segment>
+<wire x1="7.62" y1="38.1" x2="66.04" y2="38.1" width="0.1524" layer="91"/>
+<label x="10.16" y="38.1" size="1.778" layer="95"/>
 <pinref part="JP1" gate="G$1" pin="7"/>
 <pinref part="JP2" gate="G$1" pin="4"/>
-<wire x1="7.62" y1="38.1" x2="66.04" y2="38.1" width="0.1524" layer="91"/>
-<label x="10.16" y="38.1" size="1.778" layer="95"/>
 </segment>
 </net>
 <net name="RESV" class="0">
 <segment>
-<pinref part="JP2" gate="G$1" pin="5"/>
-<pinref part="JP1" gate="G$1" pin="6"/>
 <wire x1="66.04" y1="35.56" x2="7.62" y2="35.56" width="0.1524" layer="91"/>
 <label x="10.16" y="35.56" size="1.778" layer="95"/>
+<pinref part="JP1" gate="G$1" pin="6"/>
+<pinref part="JP2" gate="G$1" pin="5"/>
 </segment>
 </net>
 <net name="INCV" class="0">
 <segment>
+<wire x1="7.62" y1="33.02" x2="66.04" y2="33.02" width="0.1524" layer="91"/>
+<label x="10.16" y="33.02" size="1.778" layer="95"/>
 <pinref part="JP1" gate="G$1" pin="5"/>
 <pinref part="JP2" gate="G$1" pin="6"/>
-<wire x1="7.62" y1="33.02" x2="66.04" y2="33.02" width="0.1524" layer="91"/>
-<label x="10.16" y="33.02" size="1.778" layer="95"/>
 </segment>
 </net>
 <net name="INPHI" class="0">
 <segment>
-<pinref part="JP2" gate="G$1" pin="7"/>
-<pinref part="JP1" gate="G$1" pin="4"/>
 <wire x1="66.04" y1="30.48" x2="7.62" y2="30.48" width="0.1524" layer="91"/>
 <label x="10.16" y="30.48" size="1.778" layer="95"/>
+<pinref part="JP1" gate="G$1" pin="4"/>
+<pinref part="JP2" gate="G$1" pin="7"/>
 </segment>
 </net>
 <net name="OENABLE" class="0">
 <segment>
+<wire x1="7.62" y1="25.4" x2="66.04" y2="25.4" width="0.1524" layer="91"/>
+<label x="10.16" y="25.4" size="1.778" layer="95"/>
 <pinref part="JP1" gate="G$1" pin="2"/>
 <pinref part="JP2" gate="G$1" pin="9"/>
-<wire x1="7.62" y1="25.4" x2="66.04" y2="25.4" width="0.1524" layer="91"/>
-<label x="10.16" y="25.4" size="1.778" layer="95"/>
 </segment>
 </net>
 <net name="V_ADC" class="0">
 <segment>
-<pinref part="JP1" gate="G$1" pin="1"/>
 <wire x1="7.62" y1="22.86" x2="22.86" y2="22.86" width="0.1524" layer="91"/>
 <label x="10.16" y="22.86" size="1.778" layer="95"/>
@@
 <wire x1="43.18" y1="-5.08" x2="43.18" y2="0" width="0.1524" layer="91"/>
 <junction x="35.56" y="-5.08"/>
+<pinref part="JP1" gate="G$1" pin="1"/>
 </segment>
 <segment>
@@
 <net name="ANALOG" class="0">
 <segment>
-<pinref part="JP2" gate="G$1" pin="8"/>
 <wire x1="66.04" y1="27.94" x2="33.02" y2="27.94" width="0.1524" layer="91"/>
 <label x="55.88" y="27.94" size="1.778" layer="95"/>
@@
 <wire x1="33.02" y1="5.08" x2="33.02" y2="27.94" width="0.1524" layer="91"/>
 <label x="33.02" y="5.08" size="1.778" layer="95"/>
+<pinref part="JP2" gate="G$1" pin="8"/>
 </segment>
 </net>
 <net name="ADC-MISO" class="0">
 <segment>
-<pinref part="JP1" gate="G$1" pin="11"/>
 <wire x1="7.62" y1="48.26" x2="40.64" y2="48.26" width="0.1524" layer="91"/>
 <label x="10.16" y="48.26" size="1.778" layer="95"/>
@@
 <pinref part="U$1" gate="G$1" pin="SDATA"/>
 <wire x1="81.28" y1="2.54" x2="73.66" y2="2.54" width="0.1524" layer="91"/>
+<pinref part="JP1" gate="G$1" pin="11"/>
 </segment>
 </net>
 <net name="ADC-SCLK" class="0">
 <segment>
-<pinref part="JP1" gate="G$1" pin="12"/>
 <wire x1="7.62" y1="50.8" x2="38.1" y2="50.8" width="0.1524" layer="91"/>
 <label x="10.16" y="50.8" size="1.778" layer="95"/>
@@
 <pinref part="U$1" gate="G$1" pin="SCLK"/>
 <wire x1="83.82" y1="0" x2="73.66" y2="0" width="0.1524" layer="91"/>
+<pinref part="JP1" gate="G$1" pin="12"/>
 </segment>
 </net>
@@
 <segment>
 <pinref part="U$1" gate="G$1" pin="CS"/>
-<pinref part="JP1" gate="G$1" pin="3"/>
 <wire x1="73.66" y1="10.16" x2="73.66" y2="5.08" width="0.1524" layer="91"/>
 <wire x1="7.62" y1="27.94" x2="30.48" y2="27.94" width="0.1524" layer="91"/>
@@
 <wire x1="30.48" y1="27.94" x2="30.48" y2="10.16" width="0.1524" layer="91"/>
 <wire x1="30.48" y1="10.16" x2="73.66" y2="10.16" width="0.1524" layer="91"/>
-</segment>
-</net>
+<pinref part="JP1" gate="G$1" pin="3"/>
+</segment>
+</net>
