File: hw/pcb/impl/senseye-insight/stonyman-imager-board.sch (EAGLE design)
At the start: 8 parts, among them J1 HEADER_12PIN2X6, U1 STONYMANDEFAULT_LENS_MOUNT, U2 TI_ADCXX1S101

Commit message: updated 2X6/0.05IN headers to have no silkscreen
Parts:
- J1: value HEADER_12PIN2X6 -> HEADER_12PIN2X6_NOSILK; device senseye:HEADER_12PIN2X6 -> senseye:HEADER_12PIN2X6_NOSILK
Changed lines of the file:
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@@
 <part name="R1" library="rcl" deviceset="R-US_" device="R0603" value="0 or UNPOP"/>
 <part name="U1" library="senseye" deviceset="STONYMAN" device="DEFAULT_LENS_MOUNT"/>
-<part name="J1" library="senseye" deviceset="HEADER_12PIN" device="2X6" value="HEADER_12PIN2X6"/>
+<part name="J1" library="senseye" deviceset="HEADER_12PIN" device="2X6_NOSILK" value="HEADER_12PIN2X6_NOSILK"/>
 </parts>
 <sheets>

Commit message: added the small cap between ANALOG and GND
per Geof's suggestion.  It's an optional cap.
Parts:
- added C5: OPTIONAL: 10pF-1nF, rcl:C-EUC0603
- R1: value 0 or UNPOP -> 0 / UNPOP
Connections:
- net ANALOG: now also C5.1
- net GND: now also C5.2
Changed lines of the file:
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@@
 <part name="C3" library="rcl" deviceset="C-EU" device="C0603" value="0.1uF"/>
 <part name="C4" library="rcl" deviceset="C-EU" device="C0603" value="1uF"/>
-<part name="R1" library="rcl" deviceset="R-US_" device="R0603" value="0 or UNPOP"/>
+<part name="R1" library="rcl" deviceset="R-US_" device="R0603" value="0 / UNPOP"/>
 <part name="U1" library="senseye" deviceset="STONYMAN" device="DEFAULT_LENS_MOUNT"/>
 <part name="J1" library="senseye" deviceset="HEADER_12PIN" device="2X6_NOSILK" value="HEADER_12PIN2X6_NOSILK"/>
+<part name="C5" library="rcl" deviceset="C-EU" device="C0603" value="OPTIONAL: 10pF-1nF"/>
 </parts>
 <sheets>
@@
 <instance part="U1" gate="G$1" x="104.14" y="35.56"/>
 <instance part="J1" gate="G$1" x="106.68" y="6.35"/>
+<instance part="C5" gate="G$1" x="66.04" y="30.48" rot="R90"/>
 </instances>
 <busses>
@@
 <label x="83.82" y="12.7" size="1.778" layer="95"/>
 <pinref part="J1" gate="G$1" pin="1"/>
+<pinref part="C5" gate="G$1" pin="2"/>
+<wire x1="71.12" y1="30.48" x2="71.12" y2="25.4" width="0.1524" layer="91"/>
 </segment>
 </net>
@@
 <wire x1="33.02" y1="5.08" x2="33.02" y2="35.56" width="0.1524" layer="91"/>
 <pinref part="U1" gate="G$1" pin="ANALOG"/>
-<wire x1="33.02" y1="35.56" x2="86.36" y2="35.56" width="0.1524" layer="91"/>
+<wire x1="33.02" y1="35.56" x2="63.5" y2="35.56" width="0.1524" layer="91"/>
+<pinref part="C5" gate="G$1" pin="1"/>
+<wire x1="63.5" y1="35.56" x2="86.36" y2="35.56" width="0.1524" layer="91"/>
+<wire x1="63.5" y1="30.48" x2="63.5" y2="35.56" width="0.1524" layer="91"/>
+<junction x="63.5" y="35.56"/>
 </segment>
 </net>
