File: hw/pcb/impl/teensy-shield/main.brd (EAGLE design)
At the start: 81.9 x 19.5 mm, 37 parts, among them J1 JS202011SCQN, Q1 2N7002, Q2 2N7002, Q3 2N7002, U1 MCP73831-SOT5, U2 MAX17040-TDFN, U3 SPBT2632C2A

Commit message: removed all the stuff we're not using from board
The fuel gauge IC, the crummy camera JST connectors, everything
Parts:
- removed C3: 1uF, resistor:C0402
- removed JP6: LED, SparkFun:1X02_LOCK_LONGPADS
- removed JP7, JP8: SM08B-ZESS-TB, glasses:SM08B_8PIN_SMD
- removed Q3: 2N7002, SparkFun:SOT23-3
- removed R5: DNI, resistor:R0402
- removed U2: MAX17040-TDFN, glasses:TDFN_8PIN
Connections:
- removed net I2C_SCL: JP3.7, U2.P7
- removed net I2C_SDA: JP3.6, U2.P8
- removed net IR_LED: JP2.4, Q3.1
- removed net N$11: JP6.1, R5.1
- removed net N$12: Q3.3, R5.2
- removed net N$6: U3.P11, U3.P12
- removed net SPI_CS: JP2.3, U3.P4
- removed net SPI_MISO: JP2.1, U3.P1
- removed net SPI_MOSI: JP2.2, U3.P2
- removed net SPI_SCK: JP3.2, U3.P3
- new net CTS: JP3.7, U3.P11
- new net RTS: JP3.6, U3.P12
- new net TS_GP10: JP2.3
- new net TS_GP11: JP2.2
- new net TS_GP12: JP2.1
- new net TS_GP14: JP3.2
- new net TS_GP9: JP2.4
- net +3V3: no longer JP6.2
- net GND: no longer C3.1, JP7.P7, JP8.P2, Q3.2, U2.EP, U2.P1, U2.P4, U2.P5, U2.P6
- net INCP: no longer JP7.P2, JP8.P7
- net INCV: no longer JP7.P4, JP8.P5
- net INPHI: no longer JP7.P5, JP8.P4
- net PIXEL_EYE: no longer JP7.P8
- net PIXEL_FRONT: no longer JP8.P1
- net RESP: no longer JP7.P1, JP8.P8
- net RESV: no longer JP7.P3, JP8.P6
- net VBAT: no longer U2.P2
- net VCCIO: no longer C3.2, JP7.P6, JP8.P3, U2.P3
Routing:
- net SPI_SCK: track 83.7 -> 0.00 mm, vias 1 -> 0
- net SPI_MOSI: track 83.4 -> 0.00 mm, vias 1 -> 0
- net SPI_MISO: track 83.0 -> 0.00 mm, vias 1 -> 0
- net SPI_CS: track 81.3 -> 0.00 mm, vias 1 -> 0
- net INCV: track 47.4 -> 0.00 mm, vias 1 -> 0
- net RESV: track 46.4 -> 0.00 mm, vias 1 -> 0
- net INCP: track 45.4 -> 0.00 mm, vias 1 -> 0
- net RESP: track 44.3 -> 0.00 mm, vias 1 -> 0
- net PIXEL_EYE: track 33.8 -> 0.00 mm, vias 1 -> 0
- net VCCIO: track 111.1 -> 81.0 mm
- net PIXEL_FRONT: track 27.7 -> 0.00 mm, vias 1 -> 0
- net IR_LED: track 13.5 -> 0.00 mm
- net VBAT: track 22.6 -> 9.50 mm
- net GND: track 22.8 -> 12.7 mm
- net INPHI: track 48.4 -> 41.2 mm
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Other:
- board text removed: "498 Glasses Teensy3 Breakout"
- board text removed: "EYE"
- board text removed: "FRONT"
- board text removed: "LED"
- board text removed: "by Justin Paupore and Joe Romeo"

Commit message: finished re-routing the board
removed the stuff that wasn't used, fixing the bluetooth module's
footprint and routing RTS and CTS.
Parts:
- removed LED3: BLUE, led:CHIPLED_0603
- removed Q2: 2N7002, SparkFun:SOT23-3
- removed R4: 56, resistor:R0402
- C1, C8, C9: device resistor:C0402 -> rcl:C0603
- C2: value 1uF -> 10uF; device resistor:C0402 -> rcl:C0603
- C7: value 10uF -> 1uF
- R3: device resistor:R0402 -> rcl:R0603
- U3: device glasses:SPBT2632C2A_16PIN_SMD -> senseye:SPBT2632C2A_16PIN_SMD
- moved C10 16.5 mm to (47.9, 9.29)
- moved U3 16.5 mm to (53.7, 9.53)
- moved C4 16.5 mm to (51.3, 15.9)
- moved Q1 16.5 mm to (51.3, 13.0)
- moved C5 16.5 mm to (51.4, 9.37)
- moved R3 9.87 mm to (6.51, 13.0), turned to 0 degrees
- moved LED2 4.21 mm to (9.92, 12.9), turned to 90 degrees
- moved C1 3.20 mm to (21.2, 6.35), turned to 270 degrees
- moved C6 3.05 mm to (23.3, 6.35), turned to 270 degrees
- moved C2 2.98 mm to (21.2, 11.0)
- moved LDO1 2.86 mm to (15.6, 9.53)
- moved C7 2.82 mm to (23.3, 11.0)
- moved C9 1.11 mm to (4.45, 8.62)
- moved C8 0.64 mm to (4.45, 5.16)
- moved RESET 0.35 mm to (8.10, 5.24)
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Connections:
- removed net N$10: Q2.3, R4.2
- removed net N$8: Q2.1, U3.P5
- removed net N$9: LED3.C, R4.1
- net GND: no longer Q2.2
- net VCCIO: no longer LED3.A
Routing:
- net RTS: track 0.00 -> 56.7 mm, vias 0 -> 1
- net CTS: track 0.00 -> 55.1 mm, vias 0 -> 1
- net INPHI: track 41.2 -> 0.00 mm, vias 1 -> 0
- net UART1_TXD: track 46.6 -> 29.3 mm
- net UART1_RXD: track 41.3 -> 24.4 mm
- net VCCIO: track 81.0 -> 64.8 mm
- net N$8: track 11.7 -> 0.00 mm
- net BT_RESET: track 51.2 -> 45.0 mm
- net VIN: track 49.2 -> 51.4 mm
- net N$7: track 15.0 -> 13.0 mm
- net N$9: track 1.95 -> 0.00 mm
- net N$10: track 1.58 -> 0.00 mm
- net N$5: track 3.04 -> 1.85 mm
- net GND: track 12.7 -> 11.8 mm, vias 33 -> 25
Other:
- board size 81.9 x 19.5 mm -> 65.4 x 19.1 mm
- board text added: "SENSEYE-INSIGHT V1.1 BIELAWSKI, PAUPORE, ROMEO 5/8/2013"
- board text removed: "v1.0"
